File: esquematico_pcb/filamento_pet.kicad_pcb (KiCad board)
At the start: 2 copper layers, 17.8 x 43.2 mm, 6 parts, among them P1 Digital, P2 Analog, P3 CONN_01X01, P4 CONN_01X01, P5 CONN_01X01, P6 CONN_01X01

Commit message: Footprints elegidos
Parts:
- removed P3, P4, P5, P6: CONN_01X01, Socket_Arduino_Nano:1pin_Nano
- added A1: Pololu_A4988, Module:Pololu_Breakout-16_15.2x20.3mm, F.Cu at (116.6, 41.9)
- added C1: 100uf, Capacitor_THT:CP_Radial_D8.0mm_P3.50mm, F.Cu at (102.6, 35.6)
- added C2: 10uf, Capacitor_THT:CP_Radial_D8.0mm_P3.50mm, F.Cu at (128.5, 26.8)
- added C3: 100uf, Capacitor_THT:CP_Radial_D8.0mm_P3.50mm, F.Cu at (103.5, 22.9)
- added D1: LED, LED_THT:LED_D5.0mm, F.Cu at (100.7, 55.9)
- added D2: LED, LED_THT:LED_D5.0mm, F.Cu at (108.2, 55.9)
- added J1: 01x02M, TerminalBlock_4Ucon:TerminalBlock_4Ucon_1x02_P3.50mm_Horizontal, F.Cu at (134.0, 32.5)
- added J10: 01x03M, Connector_PinHeader_2.54mm:PinHeader_1x03_P2.54mm_Vertical, F.Cu at (38.2, 36.5)
- added J11: 01x02M, TerminalBlock_4Ucon:TerminalBlock_4Ucon_1x02_P3.50mm_Horizontal, F.Cu at (163.3, 32.5)
- added J12: 01x04M, Connector_PinHeader_2.54mm:PinHeader_1x04_P2.54mm_Vertical, F.Cu at (33.5, 26.9)
- added J13: 01x02M, TerminalBlock_4Ucon:TerminalBlock_4Ucon_1x02_P3.50mm_Horizontal, F.Cu at (163.3, 41.6)
- added J2: 01x02M, TerminalBlock_4Ucon:TerminalBlock_4Ucon_1x02_P3.50mm_Horizontal, F.Cu at (134.0, 41.6)
- added J3: 01x02M, TerminalBlock_4Ucon:TerminalBlock_4Ucon_1x02_P3.50mm_Horizontal, F.Cu at (143.8, 32.5)
- added J4: 01x02M, TerminalBlock_4Ucon:TerminalBlock_4Ucon_1x02_P3.50mm_Horizontal, F.Cu at (143.8, 41.6)
- added J5: 01x02M, TerminalBlock_4Ucon:TerminalBlock_4Ucon_1x02_P3.50mm_Horizontal, F.Cu at (153.5, 32.5)
- added J6: 01x03M, Connector_PinHeader_2.54mm:PinHeader_1x03_P2.54mm_Vertical, F.Cu at (26.9, 49.2)
- added J7: 01x03M, Connector_PinHeader_2.54mm:PinHeader_1x03_P2.54mm_Vertical, F.Cu at (31.5, 49.2)
- added J8: 01x02M, TerminalBlock_4Ucon:TerminalBlock_4Ucon_1x02_P3.50mm_Horizontal, F.Cu at (153.5, 41.6)
- added J9: 01x04M, Connector_PinHeader_2.54mm:PinHeader_1x04_P2.54mm_Vertical, F.Cu at (28.9, 26.9)
- added Q1: IRF540N, Package_TO_SOT_THT:TO-220-3_Vertical, F.Cu at (139.2, 21.3)
- added Q2: IRF540N, Package_TO_SOT_THT:TO-220-3_Vertical, F.Cu at (154.4, 20.8)
- added R1: R, Resistor_THT:R_Axial_DIN0204_L3.6mm_D1.6mm_P7.62mm_Horizontal, F.Cu at (86.1, 26.3)
- added R2: R, Resistor_THT:R_Axial_DIN0204_L3.6mm_D1.6mm_P7.62mm_Horizontal, F.Cu at (86.1, 29.5)
- added R3: R, Resistor_THT:R_Axial_DIN0204_L3.6mm_D1.6mm_P7.62mm_Horizontal, F.Cu at (86.1, 32.6)
- added R4: R, Resistor_THT:R_Axial_DIN0204_L3.6mm_D1.6mm_P7.62mm_Horizontal, F.Cu at (149.6, 53.3)
- added R5: R, Resistor_THT:R_Axial_DIN0204_L3.6mm_D1.6mm_P7.62mm_Horizontal, F.Cu at (86.1, 35.8)
- added R6: R, Resistor_THT:R_Axial_DIN0204_L3.6mm_D1.6mm_P7.62mm_Horizontal, F.Cu at (86.1, 38.9)
- added R7: R, Resistor_THT:R_Axial_DIN0204_L3.6mm_D1.6mm_P7.62mm_Horizontal, F.Cu at (86.1, 42.1)
- added R8: R, Resistor_THT:R_Axial_DIN0204_L3.6mm_D1.6mm_P7.62mm_Horizontal, F.Cu at (86.1, 45.2)
- P1, P2: footprint Socket_Arduino_Nano:Socket_Strip_Arduino_1x15 -> Connector_PinHeader_2.54mm:PinHeader_1x16_P2.54mm_Vertical
- moved P1 101.0 mm to (51.3, 21.8), turned to 0 degrees
- moved P2 98.4 mm to (69.6, 21.8), turned to 0 degrees
Connections:
- P1 pad 10: /7 -> BUT1
- P1 pad 13: /10(**/SS) -> BUT2
- P1 pad 14: /11(**/MOSI) -> BUT3
- P1 pad 5: /2 -> EN
- P1 pad 6: /3(**) -> STEP
- P1 pad 7: /4 -> DIR
- P1 pad 8: /5(**) -> MOS
- P1 pad 9: /6(**) -> FAN
- P2 pad 11: /A1 -> Pote_vel
- P2 pad 12: /A0 -> Thermistor
- P2 pad 7: /A5 -> SCL
- P2 pad 8: /A4 -> SDA
Other:
- board size 17.8 x 43.2 mm -> 150 x 50 mm
- net class Default removed
- board text removed: "1"
